File: M302N.kicad_sch (KiCad schematic)
At the start: 36 parts, among them J1 DC12V, J10 ADC_IN, J11 RJ45, J12 DC12V FAN, J13 Conn_01x05_Socket, J14 Conn_01x05_Socket, J15 Conn_01x05_Pin, J16 Conn_01x05_Pin, J17 Conn_01x08_Pin, J18 Conn_01x04_Socket, J19 Conn_01x04_Socket, J2 UART, J3 extend I/O, J4 I2C-1, J5 ADC_IN, J6 ADC_IN, J7 ADC_IN, J8 ADC_IN, J9 ADC_IN, SW1 SW_Reed, U1 W5500, U2 NJM2845DL1-05

Commit message: PCB設計中
Parts:
- R3: footprint (none) -> Varistor:RV_Disc_D12mm_W3.9mm_P7.5mm
- U2: footprint HOLLY2:NJM2845 -> Package_TO_SOT_SMD:TO-252-3_TabPin2
Connections:
- net *D10/SS: now also A1.13 (D10), J13.4 (Pin_4)
- net *D11/MOSI: now also A1.14 (D11), J13.3 (Pin_3)
- net D12/MISO: now also A1.15 (D12), J13.2 (Pin_2)
- net at J19.1 (Pin_1): now also J11.2
- net at J19.2 (Pin_2): no longer J11.6
- net at J19.3 (Pin_3): now also J11.6
- net at J18.2 (Pin_2): now also J11.3; no longer J11.2
- net at J18.3 (Pin_3): no longer J11.3
Changed lines of the file:
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@@
 	)
 	(junction
-		(at 260.35 100.33)
-		(diameter 0)
-		(color 0 0 0 0)
-	)
-	(junction
 		(at 196.85 140.97)
 		(diameter 0)
@@
 	)
 	(junction
+		(at 259.08 100.33)
+		(diameter 0)
+		(color 0 0 0 0)
+	)
+	(junction
 		(at 104.14 147.32)
 		(diameter 0)
@@
 	)
 	(no_connect
-		(at 266.7 82.55)
-	)
-	(no_connect
 		(at 269.24 82.55)
 	)
@@
 	)
 	(no_connect
-		(at 261.62 82.55)
+		(at 271.78 82.55)
 	)
 	(no_connect
@@
 	)
 	(no_connect
+		(at 264.16 82.55)
+	)
+	(no_connect
 		(at 198.12 17.78)
 	)
@@
 	(wire
 		(pts
-			(xy 260.35 100.33) (xy 260.35 102.87)
+			(xy 259.08 100.33) (xy 259.08 102.87)
 		)
 		(stroke
@@
 	(wire
 		(pts
-			(xy 264.16 82.55) (xy 264.16 105.41)
+			(xy 261.62 82.55) (xy 261.62 105.41)
 		)
 		(stroke
@@
 	(wire
 		(pts
+			(xy 261.62 105.41) (xy 257.81 105.41)
+		)
+		(stroke
+			(width 0)
+			(type default)
+		)
+	)
+	(wire
+		(pts
 			(xy 97.79 26.67) (xy 97.79 31.75)
 		)
@@
 	(wire
 		(pts
-			(xy 271.78 113.03) (xy 271.78 82.55)
+			(xy 274.32 113.03) (xy 274.32 82.55)
 		)
 		(stroke
@@
 	(wire
 		(pts
-			(xy 260.35 102.87) (xy 257.81 102.87)
+			(xy 259.08 102.87) (xy 257.81 102.87)
 		)
 		(stroke
@@
 	(wire
 		(pts
-			(xy 274.32 115.57) (xy 274.32 82.55)
+			(xy 266.7 115.57) (xy 266.7 82.55)
 		)
 		(stroke
@@
 	(wire
 		(pts
-			(xy 260.35 95.25) (xy 208.28 95.25)
+			(xy 259.08 95.25) (xy 208.28 95.25)
 		)
 		(stroke
@@
 	(wire
 		(pts
-			(xy 257.81 100.33) (xy 260.35 100.33)
+			(xy 257.81 100.33) (xy 259.08 100.33)
 		)
 		(stroke
@@
 	(wire
 		(pts
-			(xy 260.35 95.25) (xy 260.35 100.33)
+			(xy 259.08 95.25) (xy 259.08 100.33)
 		)
 		(stroke
@@
 	(wire
 		(pts
-			(xy 257.81 115.57) (xy 274.32 115.57)
+			(xy 257.81 115.57) (xy 266.7 115.57)
 		)
 		(stroke
@@
 	(wire
 		(pts
-			(xy 257.81 113.03) (xy 271.78 113.03)
+			(xy 257.81 113.03) (xy 274.32 113.03)
 		)
 		(stroke
@@
 	(wire
 		(pts
-			(xy 264.16 105.41) (xy 257.81 105.41)
-		)
-		(stroke
-			(width 0)
-			(type default)
-		)
-	)
-	(wire
-		(pts
 			(xy 172.72 91.44) (xy 177.8 91.44)
 		)
@@
 	)
 	(label "*D11{slash}MOSI"
-		(at 163.83 71.12 180)
+		(at 165.1 22.86 180)
 		(effects
 			(font
@@
 	)
 	(label "*D10{slash}SS"
-		(at 163.83 73.66 180)
+		(at 163.83 25.4 180)
 		(effects
 			(font
@@
 	)
 	(label "D12{slash}MISO"
-		(at 163.83 68.58 180)
+		(at 165.1 20.32 180)
 		(effects
 			(font
@@
 				)
 				(justify left)
+				(hide yes)
 			)
 		)
@@
 			)
 		)
-		(property "Footprint" ""
+		(property "Footprint" "Varistor:RV_Disc_D12mm_W3.9mm_P7.5mm"
 			(at 190.5 127.508 90)
 			(effects
@@
 			)
 		)
-		(property "Footprint" "HOLLY2:NJM2845"
+		(property "Footprint" "Package_TO_SOT_SMD:TO-252-3_TabPin2"
 			(at 93.98 143.51 0)
 			(effects

Commit message: もうすぐ完成
Parts:
- removed J6, J7: ADC_IN, Connector_JST:JST_XH_B3B-XH-A_1x03_P2.50mm_Vertical, symbol Connector_Generic:Conn_01x03
- added F1: LVR040, Fuse:Fuse_BelFuse_0ZRE0033FF_L11.4mm_W3.8mm, symbol Device:Polyfuse_Small
Connections:
- net +12V: now also F1.2; no longer C4.1, D3.1 (K), FL1.3, J12.2 (Pin_2)
- new net: C4.1, D3.1 (K), F1.1, FL1.3, J12.2 (Pin_2)
- no-connect marks 20 -> 22
