File: M302N.kicad_sch (KiCad schematic)
At the start: 33 parts, among them J1 DC12V, J11 RJ45, J12 DC12V FAN, J13 Conn_01x05_Socket, J14 Conn_01x05_Socket, J15 Conn_01x05_Pin, J16 Conn_01x05_Pin, J17 Conn_01x08_Pin, J18 Conn_01x04_Socket, J19 Conn_01x04_Socket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

Commit message: 階層化
Parts:
- added J8: XH-S4S, symbol Connector:Conn_01x04_Socket
- added J9: Conn_01x03_Socket, symbol Connector:Conn_01x04_Socket
Connections:
- net +5V: now also J8.2 (Pin_2)
- net GND: now also J8.1 (Pin_1)
- new net SCL: J8.4 (Pin_4)
- new net SDA: J8.3 (Pin_3)

Commit message: Soilを編集中
Parts:
- added J201: UART, symbol Connector:Conn_01x04_Socket
- J9: symbol Connector:Conn_01x04_Socket -> Connector:Conn_01x03_Socket
Connections:
- net +12V: now also C2.1, C5.1, FL1.1, U2.1 (VIN)
- net RX: now also J201.2 (Pin_2)
- net TX: now also J201.3 (Pin_3)
- net A7: now reaches J9.2 (Pin_2)
- no-connect marks 24 -> 28

Commit message: ULTRA ver 1.00
Other:
- title: M302N (under constructions) -> M302N for ULTRA
Changed lines of the file:
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@@
 	(paper "A4")
 	(title_block
-		(title "M302N (under constructions)")
-		(date "2025-05-12")
+		(title "M302N for ULTRA")
+		(date "2025-10-01")
 		(rev "2.00")
 		(company "YS-Lab Masafumi Horimoto")
