File: M302N.kicad_pcb (KiCad board)
At the start: 2 copper layers, 100.1 x 56 mm, 35 parts, among them J1 DC12V, J10 ADC_IN, J11 RJ45, J12 DC12V FAN, J13 Conn_01x05_Socket, J14 Conn_01x05_Socket, J18 Conn_01x04_Socket, J19 Conn_01x04_Socket, J2 UART, J3 extend I/O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

Commit message: もうすぐ完成
Parts:
- added F1: LVR040, Fuse:Fuse_BelFuse_0ZRE0033FF_L11.4mm_W3.8mm, F.Cu at (96.1, 72.3)
- moved D1 3.81 mm to (105.7, 74.0)
Connections:
- A1 pad 25: Net-(A1-A6) -> unconnected-(A1-A6-Pad25)
- C4 pad 1: /+12V -> Net-(D3-K)
- D3 pad 1: /+12V -> Net-(D3-K)
- FL1 pad 3: /+12V -> Net-(D3-K)
- J11 pad : GND -> (no net)
- J12 pad 2: /+12V -> Net-(D3-K)
- REF** pad 1: (no net) -> GND (x4)
Routing:
- net Net-(D3-K): track 0.00 -> 46.6 mm, vias 0 -> 1
- net /+12V: track 137.4 -> 90.9 mm, vias 2 -> 1
- net Net-(D1-A): track 15.9 -> 17.4 mm
- net Net-(J19-Pin_3): track 19.6 -> 19.1 mm
Other:
- board text added: "SCL"
- board text added: "SDA"

Commit message: PCB発注
Routing:
- net GND: track 16.6 -> 23.9 mm, vias 14 -> 9
- net /~{RESET}: track 85.7 -> 86.4 mm, vias 4 -> 3
