File: M302ULTRA/co2.kicad_sch (KiCad schematic)
At the start: 1 part, among them U501 IMG-CA0012

Commit message: ULTRA ver 1.00
Other:
- company: (none) -> YS Lab
- title: (none) -> M302N-ULTRA CO2 Sensor
Changed lines of the file:
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@@
 	(generator_version "9.0")
 	(paper "A4")
+	(title_block
+		(title "M302N-ULTRA CO2 Sensor")
+		(date "2025-10-01")
+		(rev "1.00")
+		(company "YS Lab")
+	)
 	(junction
 		(at 132.08 86.36)
