File: M302ULTRA/soil_water.kicad_sch (KiCad schematic)
At the start: 1 part, among them U601 SLT5006

Commit message: ULTRA初版・まだタイトルなし
Parts:
- added J601, J602: DIN-5, symbol Connector:DIN-5
Connections:
- net at U601. (SHIELD): now also U601.2 (GND_(BLK)), J602.2
- net at U601.1 (Vdd_(RED)): now also J602.1
- net at U601.3 (EN_(WHT)): now also J602.3
- net at U601.4 (TxD_(BLU)): now also J602.4
- net at U601.5 (RxD_(YLW)): now also J602.5
- new net +5V: J601.1, J601.3
- new net GND: J601.2
- new net RxD: J601.5
- new net TxD: J601.4
- no-connect marks 0 -> 1
Other:
- moved on the sheet: U601

Commit message: ULTRA ver 1.00
Other:
- company: (none) -> YS Lab
- title: (none) -> M302N-ULTRA Soil Water sensor
Changed lines of the file:
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@@
 	(generator_version "9.0")
 	(paper "A4")
+	(title_block
+		(title "M302N-ULTRA Soil Water sensor")
+		(date "2025-10-01")
+		(rev "1.00")
+		(company "YS Lab")
+	)
 	(junction
 		(at 96.52 95.885)
