File: M302ULTRA/temperature_humid.kicad_sch (KiCad schematic)
At the start: 1 part, among them U301 Adafruit SHT40

Commit message: ULTRA ver 1.00
Other:
- company: (none) -> YS Lab
- title: (none) -> M302N-ULTRA Temperature sensor
Changed lines of the file:
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@@
 	(generator_version "9.0")
 	(paper "A4")
+	(title_block
+		(title "M302N-ULTRA Temperature sensor")
+		(date "2025-10-01")
+		(rev "1.00")
+		(company "YS Lab")
+	)
 	(no_connect
 		(at 132.08 81.915)
