File: M302ULTRA/light_quantum.kicad_sch (KiCad schematic)
At the start: 7 parts, among them J401 DIN-3, J402 DIN-3, J403 Conn_01x10, J404 Conn_01x10_Socket, J405 Conn_01x04_Socket, U401 SQ-100X, U402 ADS1115

Commit message: ULTRA ver 1.00
Other:
- company: (none) -> YS Lab
- title: (none) -> M302N-ULTRA SQ-100X-SS
Changed lines of the file:
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@@
 	(generator_version "9.0")
 	(paper "A4")
+	(title_block
+		(title "M302N-ULTRA SQ-100X-SS")
+		(date "2025-10-01")
+		(rev "1.00")
+		(company "YS Lab")
+	)
 	(junction
 		(at 117.475 104.775)

Commit message: ULTRA ver 2.00
Parts:
- removed J403: Conn_01x10, symbol Connector_Generic:Conn_01x10
- removed J404: Conn_01x10_Socket, symbol Connector:Conn_01x06_Socket
- removed J405: Conn_01x04_Socket, symbol Connector:Conn_01x04_Socket
- removed U402: ADS1115, symbol M302N-symlib:ADS1115
Connections:
- net SIG: now reaches J401.1
- no-connect marks 5 -> 0
Other:
- moved on the sheet: J401, J402, U401
