File: M302ULTRA/M302ULTRA.kicad_sch (KiCad schematic)
At the start: 0 parts

Commit message: Soilを編集中
Parts:
- added J101: Conn_01x08_Socket, symbol Connector:Conn_01x08_Socket
- added J102: MID BOARD INTAKE, symbol Connector_Generic:Conn_01x08
- added J103: I2C-1, symbol Connector_Generic:Conn_01x04
- added J104: I2C-2, symbol Connector_Generic:Conn_01x04
- added J105: To Soil Water UNIT, symbol Connector_Generic:Conn_01x04
- added J106: To CO2 UNIT, symbol Connector_Generic:Conn_01x03
- added J107, J108, J109: Conn_01x04_Socket, symbol Connector:Conn_01x04_Socket
- added J110: Conn_01x03_Socket, symbol Connector:Conn_01x03_Socket
Connections:
- new net: J102.1 (Pin_1), J106.3 (Pin_3)
- new net: J102.2 (Pin_2), J103.1 (Pin_1), J104.1 (Pin_1), J105.1 (Pin_1), J106.1 (Pin_1)
- new net: J102.3 (Pin_3), J103.2 (Pin_2), J104.2 (Pin_2), J105.4 (Pin_4)
- new net: J102.4 (Pin_4), J103.4 (Pin_4), J104.4 (Pin_4)
- new net: J102.5 (Pin_5), J103.3 (Pin_3), J104.3 (Pin_3)
- new net: J102.6 (Pin_6), J105.3 (Pin_3)
- new net: J102.7 (Pin_7), J105.2 (Pin_2)
- new net: J102.8 (Pin_8), J106.2 (Pin_2)
- new net CO2/+12V: J110.3 (Pin_3)
- new net CO2/GND: J110.1 (Pin_1)
- new net CO2/OUT: J110.2 (Pin_2)
- new net Light Quantum/+5V: J108.2 (Pin_2)
- new net Light Quantum/GND: J108.1 (Pin_1)
- new net Light Quantum/SCL: J108.4 (Pin_4)
- new net Light Quantum/SDA: J108.3 (Pin_3)
- new net M302N_CPU/+12V: J101.1 (Pin_1)
- new net M302N_CPU/+5V: J101.3 (Pin_3)
- new net M302N_CPU/A7: J101.8 (Pin_8)
- new net M302N_CPU/GND: J101.2 (Pin_2)
- new net M302N_CPU/RX: J101.7 (Pin_7)
- new net M302N_CPU/SCL: J101.4 (Pin_4)
- new net M302N_CPU/SDA: J101.5 (Pin_5)
- new net M302N_CPU/TX: J101.6 (Pin_6)
- new net Temperature and Humid/+5V: J107.2 (Pin_2)
- new net Temperature and Humid/GND: J107.1 (Pin_1)
- new net Temperature and Humid/SCL: J107.4 (Pin_4)
- new net Temperature and Humid/SDA: J107.3 (Pin_3)
Other:
- added sheet CO2 (co2.kicad_sch)
- added sheet Light Quantum (light_quantum.kicad_sch)
- added sheet Soil Water (soil_water.kicad_sch)
- added sheet Temperature and Humid (temperature_humid.kicad_sch)
- sheet M302N_CPU ports: added +12V, +5V, A7, GND, RX, SCL, SDA, TX; removed none
- note added: "CO2 UNIT IMG-CA0012"
- note added: "LIGHT QUANTUM UNIT SQ-100X ADS1115"
- note added: "M302N CPU UNIT"
- note added: "SOIL WATER UNIT SLT-5006"
- note added: "TEMPERATURE HUMIDITY UNIT SHT-40"

Commit message: ULTRA初版・まだタイトルなし
Connections:
- net Soil Water/GND: now reaches J109.1 (Pin_1)
- net Soil Water/TxD: now reaches J109.2 (Pin_2)
- net Soil Water/RxD: now reaches J109.3 (Pin_3)
- net Soil Water/+5V: now reaches J109.4 (Pin_4)
Other:
- sheet Soil Water ports: added +5V, GND, RxD, TxD; removed none
Changed lines of the file:
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@@
 	(text "CO2 UNIT\nIMG-CA0012"
 		(exclude_from_sim no)
-		(at 162.56 137.795 0)
+		(at 163.195 141.605 0)
 		(effects
 			(font
@@
 	(text "SOIL WATER UNIT\nSLT-5006"
 		(exclude_from_sim no)
-		(at 203.2 137.795 0)
+		(at 202.565 141.605 0)
 		(effects
 			(font
@@
 	(wire
 		(pts
+			(xy 186.69 113.03) (xy 186.69 127.635)
+		)
+		(stroke
+			(width 0)
+			(type default)
+		)
+	)
+	(wire
+		(pts
 			(xy 84.455 64.135) (xy 109.22 64.135)
 		)
@@
 	(wire
 		(pts
+			(xy 191.77 113.03) (xy 191.77 127.635)
+		)
+		(stroke
+			(width 0)
+			(type default)
+		)
+	)
+	(wire
+		(pts
 			(xy 75.565 64.135) (xy 84.455 64.135)
 		)
@@
 	(wire
 		(pts
+			(xy 189.23 113.03) (xy 189.23 127.635)
+		)
+		(stroke
+			(width 0)
+			(type default)
+		)
+	)
+	(wire
+		(pts
 			(xy 86.995 93.345) (xy 86.995 61.595)
 		)
@@
 		(pts
 			(xy 84.455 90.805) (xy 64.77 90.805)
+		)
+		(stroke
+			(width 0)
+			(type default)
+		)
+	)
+	(wire
+		(pts
+			(xy 194.31 113.03) (xy 194.31 127.635)
 		)
 		(stroke
@@
 			)
 		)
+		(pin "+5V" input
+			(at 186.69 127.635 90)
+			(effects
+				(font
+					(size 1.27 1.27)
+				)
+				(justify right)
+			)
+		)
+		(pin "GND" input
+			(at 194.31 127.635 90)
+			(effects
+				(font
+					(size 1.27 1.27)
+				)
+				(justify right)
+			)
+		)
+		(pin "RxD" input
+			(at 189.23 127.635 90)
+			(effects
+				(font
+					(size 1.27 1.27)
+				)
+				(justify right)
+			)
+		)
+		(pin "TxD" output
+			(at 191.77 127.635 90)
+			(effects
+				(font
+					(size 1.27 1.27)
+				)
+				(justify right)
+			)
+		)

Commit message: 外観デザインスケッチを追加
Parts:
- J101: value Conn_01x08_Socket -> XHP8
- J107, J108, J109: value Conn_01x04_Socket -> XHP4
- J110: value Conn_01x03_Socket -> XHP3
Changed lines of the file:
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@@
 		(dnp no)
 		(property "Reference" "J107"
-			(at 52.705 109.855 90)
-			(effects
-				(font
-					(size 1.27 1.27)
-				)
-			)
-		)
-		(property "Value" "Conn_01x04_Socket"
-			(at 52.705 112.2793 90)
+			(at 59.055 109.22 90)
+			(effects
+				(font
+					(size 1.27 1.27)
+				)
+			)
+		)
+		(property "Value" "XHP4"
+			(at 59.055 111.6443 90)
 			(effects
 				(font
@@
 			)
 		)
-		(property "Value" "Conn_01x08_Socket"
-			(at 44.45 75.565 0)
+		(property "Value" "XHP8"
+			(at 60.325 73.66 0)
 			(effects
 				(font
@@
 		(dnp no)
 		(property "Reference" "J110"
-			(at 165.735 109.3357 90)
-			(effects
-				(font
-					(size 1.27 1.27)
-				)
-			)
-		)
-		(property "Value" "Conn_01x03_Socket"
-			(at 165.735 111.76 90)
+			(at 142.24 108.585 90)
+			(effects
+				(font
+					(size 1.27 1.27)
+				)
+			)
+		)
+		(property "Value" "XHP3"
+			(at 142.24 111.0093 90)
 			(effects
 				(font
@@
 		(dnp no)
 		(property "Reference" "J108"
-			(at 97.155 109.9707 90)
-			(effects
-				(font
-					(size 1.27 1.27)
-				)
-			)
-		)
-		(property "Value" "Conn_01x04_Socket"
-			(at 97.155 112.395 90)
+			(at 102.87 108.7007 90)
+			(effects
+				(font
+					(size 1.27 1.27)
+				)
+			)
+		)
+		(property "Value" "XHP4"
+			(at 102.87 111.125 90)
 			(effects
 				(font
@@
 		(dnp no)
 		(property "Reference" "J109"
-			(at 205.105 109.3357 90)
-			(effects
-				(font
-					(size 1.27 1.27)
-				)
-			)
-		)
-		(property "Value" "Conn_01x04_Socket"
-			(at 205.105 111.76 90)
+			(at 179.705 108.585 90)
+			(effects
+				(font
+					(size 1.27 1.27)
+				)
+			)
+		)
+		(property "Value" "XHP4"
+			(at 179.705 111.0093 90)
 			(effects
 				(font
@@
 			)
 		)
-		(pin "SCL" output
+		(pin "SCL" bidirectional
 			(at 47.625 48.895 270)
 			(effects
@@
 			)
 		)
-		(pin "SDA" output
+		(pin "SDA" bidirectional
 			(at 49.53 48.895 270)
 			(effects

Commit message: ULTRA ver 1.00
Other:
- company: (none) -> YS Lab
- title: (none) -> M302N-ULTRA for Green HOUSE
Changed lines of the file:
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@@
 	(generator_version "9.0")
 	(paper "A4")
+	(title_block
+		(title "M302N-ULTRA for Green HOUSE")
+		(date "2025-10-01")
+		(rev "1.00")
+		(company "YS Lab")
+	)
 	(text "TEMPERATURE\nHUMIDITY\nUNIT\nSHT-40"
 		(exclude_from_sim no)

Commit message: ULTRA ver 2.00
Parts:
- removed J104: I2C-2, symbol Connector_Generic:Conn_01x04
- added J10: AIN0, symbol Connector_Generic:Conn_01x02
- added J20: AIN1, symbol Connector_Generic:Conn_01x02
- added J21: AIN2, symbol Connector_Generic:Conn_01x02
- added J22: AIN3, symbol Connector_Generic:Conn_01x02
- added U3: ADS1115, symbol M302N:ADS1115
- J108: symbol Connector:Conn_01x04_Socket -> Connector:Conn_01x02_Socket
Connections:
- net at J102.2 (Pin_2), J103.1 (Pin_1), J105.1 (Pin_1)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: now also J10.1 (Pin_1), J20.1 (Pin_1), J21.1 (Pin_1), J22.1 (Pin_1), U3.2 (GND)
- net at J102.3 (Pin_3), J103.2 (Pin_2), J105.4 (Pin_4): now also U3.1 (VDD)
- net at J102.4 (Pin_4), J103.4 (Pin_4): now also U3.3 (SCL)
- net at J102.5 (Pin_5), J103.3 (Pin_3): now also U3.4 (SDA)
- net Light Quantum/+5V renamed Light Quantum/SIG
- removed net Light Quantum/SCL: J108.4 (Pin_4)
- removed net Light Quantum/SDA: J108.3 (Pin_3)
- new net: J22.2 (Pin_2), U3.10 (AIN3)
- new net: J10.2 (Pin_2), U3.7 (AIN0)
- new net: J21.2 (Pin_2), U3.9 (AIN2)
- new net: J20.2 (Pin_2), U3.8 (AIN1)
- no-connect marks 0 -> 2
Other:
- sheet Light Quantum ports: added SIG; removed +5V, SCL, SDA
- moved on the sheet: J105, J106, J109, J110

Commit message: Ver 2.10 Append DDS
Parts:
- added FL101: 0.1uF DDS1, HOLLY2:DSS1, symbol 001-rescue:EMI_Filter_LCL-Device
Connections:
- net at J10.1 (Pin_1), J102.2 (Pin_2), J103.1 (Pin_1)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: now also FL101.2
- net at J102.1 (Pin_1): now also FL101.1; no longer J106.3 (Pin_3)
- new net: FL101.3, J106.3 (Pin_3)
Changed lines of the file:
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@@
 		(title "M302N-ULTRA for Green HOUSE")
 		(date "2025-10-01")
-		(rev "2.00")
+		(rev "2.10")
 		(company "YS Lab")
+		(comment 1 "Append DDS1")
 	)
 	(text "TEMPERATURE\nHUMIDITY\nUNIT\nSHT-40"
@@
 	)
 	(junction
+		(at 186.69 85.09)
+		(diameter 0)
+		(color 0 0 0 0)
+	)
+	(junction
 		(at 116.84 106.045)
 		(diameter 0)
@@
 	(wire
 		(pts
+			(xy 186.69 85.09) (xy 186.69 97.79)
+		)
+		(stroke
+			(width 0)
+			(type default)
+		)
+	)
+	(wire
+		(pts
 			(xy 134.62 96.52) (xy 127 96.52)
 		)
@@
 	(wire
 		(pts
+			(xy 181.61 95.885) (xy 181.61 97.79)
+		)
+		(stroke
+			(width 0)
+			(type default)
+		)
+	)
+	(wire
+		(pts
 			(xy 129.54 99.06) (xy 129.54 109.855)
 		)
@@
 	(wire
 		(pts
-			(xy 181.61 71.755) (xy 181.61 97.79)
+			(xy 182.245 85.09) (xy 186.69 85.09)
+		)
+		(stroke
+			(width 0)
+			(type default)
+		)
+	)
+	(wire
+		(pts
+			(xy 177.165 71.755) (xy 177.165 77.47)
 		)
 		(stroke
@@
 	(wire
 		(pts
+			(xy 177.165 95.885) (xy 181.61 95.885)
+		)
+		(stroke
+			(width 0)
+			(type default)
+		)
+	)
+	(wire
+		(pts
 			(xy 67.945 113.03) (xy 67.945 127)
 		)
@@
 	(wire
 		(pts
-			(xy 186.69 69.215) (xy 186.69 97.79)
+			(xy 186.69 69.215) (xy 186.69 85.09)
 		)
 		(stroke
@@
 	(wire
 		(pts
+			(xy 177.165 92.71) (xy 177.165 95.885)
+		)
+		(stroke
+			(width 0)
+			(type default)
+		)
+	)
+	(wire
+		(pts
 			(xy 43.815 69.215) (xy 60.325 69.215)
 		)
@@
 	(wire
 		(pts
-			(xy 75.565 71.755) (xy 181.61 71.755)
+			(xy 75.565 71.755) (xy 177.165 71.755)
 		)
 		(stroke
@@
 					(unit 1)
 				)
+			)
+		)
+	)
+	(symbol
+		(lib_id "001-rescue:EMI_Filter_LCL-Device")
+		(at 179.705 85.09 90)
+		(mirror x)
+		(unit 1)
+		(exclude_from_sim no)
+		(in_bom yes)
+		(on_board yes)
+		(dnp no)
+		(property "Reference" "FL101"
+			(at 171.6532 85.09 0)
+			(effects
+				(font
+					(size 1.27 1.27)
+				)
+			)
+		)
+		(property "Value" "0.1uF DDS1"
+			(at 173.9646 85.09 0)
+			(effects
+				(font
+					(size 1.27 1.27)
+				)
+			)
+		)
+		(property "Footprint" "HOLLY2:DSS1"
+			(at 179.705 85.09 90)
+			(effects
+				(font
+					(size 1.27 1.27)
+				)
+				(hide yes)
+			)
+		)
+		(property "Datasheet" "http://www.murata.com/~/media/webrenewal/support/library/catalog/products/emc/emifil/c31e.ashx?la=en-gb"
+			(at 179.705 85.09 90)
+			(effects
+				(font
+					(size 1.27 1.27)
+				)
+				(hide yes)
+			)
+		)
+		(property "Description" ""
+			(at 179.705 85.09 0)
+			(effects
+				(font
+					(size 1.27 1.27)
+				)
+				(hide yes)
+			)
+		)
+		(pin "1"
+		)
+		(pin "3"
+		)
+		(pin "2"
+		)
+		(instances
+			(project "M302ULTRA"
+				(path "/d9d02f3f-e7de-4839-b3af-9017ce7335aa"
+					(reference "FL101")
+					(unit 1)
+				)
